File: hw/design/HR_SENSOR.sch (KiCad schematic (older format))
At the start: 6 parts

Commit message: Slow day for the project, wasn't really feeling inspired.
Actually quite tilted that 0 keypad switch manufacturers offer schematic
symbols and footprints of their products.

Oh well, added uUSB traces and moves the sheets around to prepare for PMU
integration.

It's also painfully obvious that there's a lot to do for parts I have already
traced; I need to make sure current, voltage, etc. are all in line with specs
for every piece. Kinda feels like I have made big strides already, but I am not
ready to stop.
Connections:
- net HR1V8 renamed HR_1V8
- net HR3V3 renamed HR_3V3
Changed lines of the file:
@@
 	4700 4550 4700 5000
 Connection ~ 4700 4550
-Text GLabel 4700 5000 3    50   Input ~ 0
-HR1V8
 Wire Wire Line
 	4550 2900 4550 3800
@@
 Wire Wire Line
 	6750 4700 6950 4700
-Text GLabel 4550 2200 1    50   Input ~ 0
-VDDIO
 Wire Wire Line
 	4550 2400 4550 2200
@@
 	7000 3650 7000 3200
 Connection ~ 7000 3650
-Text GLabel 7000 3200 1    50   Input ~ 0
-HR3V3
 Wire Wire Line
 	7000 3800 7000 3650
@@
 Text HLabel 5050 2900 2    50   Output ~ 0
 HR_INT
+Text HLabel 4550 2200 1    50   Input ~ 0
+VDDIO
+Text HLabel 7000 3200 1    50   Input ~ 0
+HR_3V3
+Text HLabel 4700 5000 3    50   Input ~ 0
+HR_1V8
 $EndSCHEMATC
