File: hw/design/MCU_V.sch (KiCad schematic (older format))
At the start: 1 part

Commit message: Slow day for the project, wasn't really feeling inspired.
Actually quite tilted that 0 keypad switch manufacturers offer schematic
symbols and footprints of their products.

Oh well, added uUSB traces and moves the sheets around to prepare for PMU
integration.

It's also painfully obvious that there's a lot to do for parts I have already
traced; I need to make sure current, voltage, etc. are all in line with specs
for every piece. Kinda feels like I have made big strides already, but I am not
ready to stop.
Connections:
- net VDDIO1: now reaches U?.A5 (VDDIO)
Changed lines of the file:
@@
 $Descr A4 11693 8268
 encoding utf-8
-Sheet 4 7
+Sheet 3 7
 Title ""
 Date ""
@@
 	1    0    0    -1
 $EndComp
+Wire Wire Line
+	4825 3650 4200 3650
+Text HLabel 4200 3650 0    50   Output ~ 0
+VDDIO1
 $EndSCHEMATC
