File: hw/design/design.sch (KiCad schematic (older format))
At the start: 0 parts

Commit message: Slow day for the project, wasn't really feeling inspired.
Actually quite tilted that 0 keypad switch manufacturers offer schematic
symbols and footprints of their products.

Oh well, added uUSB traces and moves the sheets around to prepare for PMU
integration.

It's also painfully obvious that there's a lot to do for parts I have already
traced; I need to make sure current, voltage, etc. are all in line with specs
for every piece. Kinda feels like I have made big strides already, but I am not
ready to stop.
Changed lines of the file:
@@
 $EndDescr
 $Sheet
-S 1950 1250 700  550
+S 3725 1225 700  550
 U 5E0A3409
 F0 "HR Sensor" 50
 F1 "HR_SENSOR.sch" 50
-F2 "HR_SDA" B R 2650 1400 50
-F3 "HR_SCL" I R 2650 1500 50
-F4 "HR_INT" O R 2650 1600 50
+F2 "HR_SDA" B R 4425 1275 50
+F3 "HR_SCL" I R 4425 1375 50
+F4 "HR_INT" O R 4425 1475 50
+F5 "VDDIO" I R 4425 1600 50
+F6 "HR_3V3" I L 3725 1725 50
+F7 "HR_1V8" I L 3725 1650 50
 $EndSheet
 Wire Wire Line
-	2650 1400 4100 1400
+	4425 1275 5875 1275
 Wire Wire Line
-	4100 1500 2650 1500
+	5875 1375 4425 1375
 Wire Wire Line
-	2650 1600 4100 1600
+	4425 1475 5875 1475
 $Sheet
-S 8050 1475 900  1450
+S 1825 1200 900  1450
 U 5E15CBF8
 F0 "MCU Power" 50
 F1 "MCU_V.sch" 50
+F2 "VDDIO1" O R 2725 2125 50
 $EndSheet
 $Sheet
-S 9350 1475 700  750
+S 4875 5050 700  750
 U 5E17C70B
 F0 "MCU Peripherals" 50
 F1 "MCU_Peripherals.sch" 50
+F2 "DM" B R 5575 5200 50
+F3 "DP" B R 5575 5300 50
 $EndSheet
 $Sheet
-S 2825 2975 550  850
+S 4600 2850 550  850
 U 5E180B58
 F0 "SD Card" 50
 F1 "SD_Card.sch" 50
-F2 "SD_DAT1" B R 3375 3100 50
-F3 "SD_DAT0" B R 3375 3025 50
-F4 "SD_DAT2" B R 3375 3175 50
-F5 "SD_DAT3" B R 3375 3250 50
-F6 "SD_CMD" I R 3375 3375 50
-F7 "SD_CLK" I R 3375 3450 50
-F9 "SD_SW" O R 3375 3575 50
+F2 "SD_DAT1" B R 5150 2975 50
+F3 "SD_DAT0" B R 5150 2900 50
+F4 "SD_DAT2" B R 5150 3050 50
+F5 "SD_DAT3" B R 5150 3125 50
+F6 "SD_CMD" I R 5150 3250 50
+F7 "SD_CLK" I R 5150 3325 50
+F8 "SD_SW" O R 5150 3450 50
 $EndSheet
 $Sheet
-S 4100 1300 1150 2825
+S 5875 1175 1150 2825
 U 5E117560
 F0 "MCU GPIO" 50
 F1 "MCU_GPIO.sch" 50
-F2 "HR_INT_GPIO" I L 4100 1600 50
-F3 "I2C1_SDA" B L 4100 1400 50
-F4 "I2C1_SCL" O L 4100 1500 50
-F5 "SD_SW_GPIO" I L 4100 3575 50
-F6 "SDHC_DAT0" B L 4100 3025 50
-F7 "SDHC_CLK" O L 4100 3450 50
-F8 "SDHC_DAT1" B L 4100 3100 50
-F9 "SDHC_DAT3" B L 4100 3250 50
-F10 "SDHC_CMD" O L 4100 3375 50
-F11 "SDHC_DAT2" B L 4100 3175 50
+F2 "HR_INT_GPIO" I L 5875 1475 50
+F3 "I2C1_SDA" B L 5875 1275 50
+F4 "I2C1_SCL" O L 5875 1375 50
+F5 "SD_SW_GPIO" I L 5875 3450 50
+F6 "SDHC_DAT0" B L 5875 2900 50
+F7 "SDHC_CLK" O L 5875 3325 50
+F8 "SDHC_DAT1" B L 5875 2975 50
+F9 "SDHC_DAT3" B L 5875 3125 50
+F10 "SDHC_CMD" O L 5875 3250 50
+F11 "SDHC_DAT2" B L 5875 3050 50
 $EndSheet
 Wire Wire Line
-	4100 3025 3375 3025
+	5875 2900 5150 2900
 Wire Wire Line
-	3375 3100 4100 3100
+	5150 2975 5875 2975
 Wire Wire Line
-	4100 3175 3375 3175
+	5875 3050 5150 3050
 Wire Wire Line
-	3375 3250 4100 3250
+	5150 3125 5875 3125
 Wire Wire Line
-	3375 3375 4100 3375
+	5150 3250 5875 3250
 Wire Wire Line
-	3375 3450 4100 3450
+	5150 3325 5875 3325
 Wire Wire Line
-	3375 3575 4100 3575
+	5150 3450 5875 3450
 $Sheet
-S 6150 1325 500  325
+S 6275 5125 500  325
 U 5E1BF042
 F0 "Micro USB" 50
 F1 "uUSB.sch" 50
+F2 "D-" B L 6275 5200 50
+F3 "D+" B L 6275 5300 50
+F4 "VCC" O R 6775 5250 50
 $EndSheet
+Wire Wire Line
+	6275 5200 5575 5200
+Wire Wire Line
+	6275 5300 5575 5300
+Wire Wire Line
+	4425 1600 4625 1600
+Wire Wire Line
+	4625 1600 4625 2125
+Wire Wire Line
+	4625 2125 2725 2125
 $EndSCHEMATC
