File: hw/design/uUSB.sch (KiCad schematic (older format))
At the start: 1 part

Commit message: Slow day for the project, wasn't really feeling inspired.
Actually quite tilted that 0 keypad switch manufacturers offer schematic
symbols and footprints of their products.

Oh well, added uUSB traces and moves the sheets around to prepare for PMU
integration.

It's also painfully obvious that there's a lot to do for parts I have already
traced; I need to make sure current, voltage, etc. are all in line with specs
for every piece. Kinda feels like I have made big strides already, but I am not
ready to stop.
Connections:
- net VCC: now reaches J?.1
- net D-: now reaches J?.2
- net D+: now reaches J?.3
- net GND: now reaches J?.4
- net GND: now also J?.5, J?.SH
Changed lines of the file:
@@
 	1    0    0    -1
 $EndComp
+Wire Wire Line
+	5650 4150 5650 4200
+$Comp
+L power:GND #PWR?
+U 1 1 5DFD685B
+P 5650 4400
+F 0 "#PWR?" H 5650 4150 50  0001 C CNN
+F 1 "GND" H 5655 4227 50  0000 C CNN
+F 2 "" H 5650 4400 50  0001 C CNN
+F 3 "" H 5650 4400 50  0001 C CNN
+	1    5650 4400
+	1    0    0    -1
+$EndComp
+Wire Wire Line
+	6050 3350 6350 3350
+Wire Wire Line
+	6350 3350 6350 3000
+Wire Wire Line
+	6050 3450 6500 3450
+Wire Wire Line
+	6050 3550 6500 3550
+Wire Wire Line
+	6050 3750 6050 4200
+Wire Wire Line
+	6050 4200 5650 4200
+Connection ~ 5650 4200
+Wire Wire Line
+	5650 4200 5650 4400
+Wire Wire Line
+	6050 3650 6150 3650
+Wire Wire Line
+	6150 3650 6150 4200
+Wire Wire Line
+	6150 4200 6050 4200
+Connection ~ 6050 4200
+Text HLabel 6500 3450 2    50   BiDi ~ 0
+D-
+Text HLabel 6500 3550 2    50   BiDi ~ 0
+D+
+Text HLabel 6350 3000 1    50   Output ~ 0
+VCC
 $EndSCHEMATC
